Commit message: update

File: src/robot_properties/urdf/controllers/omni_drive.urdf.xacro (robot description, xacro)
@@ -2,5 +2,5 @@
   <xacro:macro name="omni_drive_controller">
     <gazebo>
-      <plugin name="object_controller" filename="libgazebo_ros_planar_move.so">
+      <plugin name="omni_controller" filename="libgazebo_ros_planar_move.so">
         <ros>
           <remapping>odom:=odom/unfiltered</remapping>

File: src/robot_properties/urdf/robots/robot.urdf.xacro (robot description, xacro)
@@ -9,8 +9,12 @@
   <xacro:include filename="$(find robot_properties)/urdf/controllers/omni_drive.urdf.xacro" />
   <xacro:include filename="$(find ur_description)/urdf/ur_macro.xacro" />
-   <!-- initial position for simulations (Fake Hardware, Gazebo, Ignition) -->
-   <xacro:arg name="arm_initial_positions_file" default="$(find robot_properties)/config/arm_initial_positions.yaml"/>
-   <!-- convert to property to use substitution in function -->
-   <xacro:property name="arm_initial_positions_file" default="$(arg arm_initial_positions_file)"/>
+  <!-- <xacro:include filename="$(find ur_description)/urdf/inc/ur_joint_control.xacro" /> -->
+  <!-- <xacro:include filename="$(find ur_description)/urdf/inc/ur_sensors.xacro" /> -->
+  <!-- initial position for simulations (Fake Hardware, Gazebo, Ignition) -->
+  <xacro:arg name="arm_initial_positions_file"
+    default="$(find robot_properties)/config/arm_initial_positions.yaml" />
+  <!-- convert to property to use substitution in function -->
+  <xacro:property name="arm_initial_positions_file"
+    default="$(arg arm_initial_positions_file)" />
   <!-- UR arm mounted on mobile base -->
   <xacro:if value="$(arg use_arm)">
@@ -23,10 +27,11 @@
       physical_parameters_file="$(find ur_description)/config/ur5/physical_parameters.yaml"
       visual_parameters_file="$(find ur_description)/config/ur5/visual_parameters.yaml"
+      generate_ros2_control_tag="true"
       transmission_hw_interface="hardware_interface/PositionJointInterface"
+      use_fake_hardware="true"
       safety_limits="true"
       safety_pos_margin="0.15"
       safety_k_position="20"
       sim_gazebo="true"
-      use_fake_hardware="true"
       initial_positions="${xacro.load_yaml(arm_initial_positions_file)}"
     >
